File: tamagotya.sch (EAGLE design)
At the start: 67 parts, among them U1 ADXL345, U100 ESP32-D2WD, U1000 TP4056, U1500 FS312F-G, U1550 FS8205, U200 UT-0206-P05FOLDED, U2000 MT3608, U2100 M3406, U300 4MB Flash, Y100 40Mhz 3.2X2.5

Commit message: Add a NPN transitor to drive a piezo speaker
Parts:
- added PIEZO+, PIEZO-: WIREPADSMD1,27-254, wirepad:WIREPADSMD1,27-254
- added Q1: 600mA/40V, SparkFun-DiscreteSemi:TRANS_NPN-MMBT2222AL
- added R6: 1k, rcl:R-EU_R0603
Connections:
- new net N$5: Q1.B, R6.2
- new net PIEZO_GND: PIEZO-.P, Q1.C
- net 5V: now also PIEZO+.P
- net GND: now also Q1.E
- net GPIO14: now also R6.1
Changed lines of the file:
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@@
 <part name="SUPPLY22" library="SparkFun-PowerSymbols" library_urn="urn:adsk.eagle:library:530" deviceset="V_BATT" device=""/>
 <part name="GND31" library="SparkFun-PowerSymbols" library_urn="urn:adsk.eagle:library:530" deviceset="GND" device=""/>
+<part name="PIEZO+" library="wirepad" library_urn="urn:adsk.eagle:library:412" deviceset="WIREPAD" device="SMD1,27-254" package3d_urn="urn:adsk.eagle:package:30839/1"/>
+<part name="PIEZO-" library="wirepad" library_urn="urn:adsk.eagle:library:412" deviceset="WIREPAD" device="SMD1,27-254" package3d_urn="urn:adsk.eagle:package:30839/1"/>
+<part name="SUPPLY23" library="SparkFun-PowerSymbols" deviceset="5V" device=""/>
+<part name="Q1" library="SparkFun-DiscreteSemi" deviceset="TRANS_NPN" device="-MMBT2222AL" value="600mA/40V"/>
+<part name="GND32" library="SparkFun-PowerSymbols" library_urn="urn:adsk.eagle:library:530" deviceset="GND" device=""/>
+<part name="R6" library="rcl" library_urn="urn:adsk.eagle:library:334" deviceset="R-EU_" device="R0603" package3d_urn="urn:adsk.eagle:package:23555/2" value="1k"/>
 </parts>
 <sheets>
@@
 <instance part="SUPPLY20" gate="G$1" x="147.32" y="152.4" smashed="yes">
 <attribute name="VALUE" x="147.32" y="155.194" size="1.778" layer="96" align="bottom-center"/>
+</instance>
+<instance part="PIEZO+" gate="G$1" x="81.28" y="170.18" smashed="yes">
+<attribute name="NAME" x="80.137" y="172.0342" size="1.778" layer="95"/>
+</instance>
+<instance part="PIEZO-" gate="G$1" x="81.28" y="162.56" smashed="yes">
+<attribute name="NAME" x="80.137" y="164.4142" size="1.778" layer="95"/>
+</instance>
+<instance part="SUPPLY23" gate="G$1" x="96.52" y="172.72" smashed="yes">
+<attribute name="VALUE" x="96.52" y="175.514" size="1.778" layer="96" align="bottom-center"/>
+</instance>
+<instance part="Q1" gate="G$1" x="93.98" y="154.94" smashed="yes">
+<attribute name="NAME" x="96.52" y="154.94" size="1.778" layer="95" font="vector"/>
+<attribute name="VALUE" x="96.52" y="152.654" size="1.778" layer="96" font="vector"/>
+</instance>
+<instance part="GND32" gate="1" x="96.52" y="144.78" smashed="yes">
+<attribute name="VALUE" x="96.52" y="144.526" size="1.778" layer="96" align="top-center"/>
+</instance>
+<instance part="R6" gate="G$1" x="83.82" y="154.94" smashed="yes">
+<attribute name="NAME" x="80.01" y="156.4386" size="1.778" layer="95"/>
+<attribute name="VALUE" x="80.01" y="151.638" size="1.778" layer="96"/>
 </instance>
 </instances>
@@
 <pinref part="GND30" gate="1" pin="GND"/>
 </segment>
+<segment>
+<pinref part="Q1" gate="G$1" pin="E"/>
+<wire x1="96.52" y1="149.86" x2="96.52" y2="147.32" width="0.1524" layer="91"/>
+<pinref part="GND32" gate="1" pin="GND"/>
+</segment>
 </net>
 <net name="GPIO16" class="0">
@@
 <label x="63.5" y="30.48" size="1.27" layer="95" rot="R270" xref="yes"/>
 </segment>
+<segment>
+<pinref part="R6" gate="G$1" pin="1"/>
+<wire x1="78.74" y1="154.94" x2="76.2" y2="154.94" width="0.1524" layer="91"/>
+<label x="76.2" y="154.94" size="1.27" layer="95" rot="R180" xref="yes"/>
+</segment>
 </net>
 <net name="GPIO12" class="0">
@@
 </segment>
 </net>
+<net name="PIEZO_GND" class="0">
+<segment>
+<pinref part="PIEZO-" gate="G$1" pin="P"/>
+<wire x1="83.82" y1="162.56" x2="96.52" y2="162.56" width="0.1524" layer="91"/>
+<pinref part="Q1" gate="G$1" pin="C"/>
+<wire x1="96.52" y1="160.02" x2="96.52" y2="162.56" width="0.1524" layer="91"/>
+<label x="96.52" y="162.56" size="1.27" layer="95" xref="yes"/>
+</segment>
+</net>
+<net name="5V" class="0">
+<segment>
+<pinref part="PIEZO+" gate="G$1" pin="P"/>
+<wire x1="83.82" y1="170.18" x2="96.52" y2="170.18" width="0.1524" layer="91"/>
+<wire x1="96.52" y1="170.18" x2="96.52" y2="172.72" width="0.1524" layer="91"/>
+<pinref part="SUPPLY23" gate="G$1" pin="5V"/>
+</segment>
+</net>
+<net name="N$5" class="0">
+<segment>
+<pinref part="Q1" gate="G$1" pin="B"/>
+<wire x1="91.44" y1="154.94" x2="88.9" y2="154.94" width="0.1524" layer="91"/>
+<pinref part="R6" gate="G$1" pin="2"/>
+</segment>
+</net>
