File: tamagotya.brd (EAGLE design)
At the start: 27.9 x 31.8 mm, 71 parts, among them Q1 600mA/40V, U1 ADXL345, U100 ESP32-D2WD, U1000 TP4056, U1500 FS312F-G, U1550 FS8205, U200 UT-0206-P05FOLDED, U2000 MT3608, U2100 M3406, U300 4MB Flash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

Commit message: Fix collision between antenna and switch holes
Parts:
- moved E1 1.14 mm to (17.0, 5.21)
- moved U$3 0.25 mm to (24.0, 3.94)
- moved C4 0.25 mm to (22.9, 3.81)
- moved R3 0.25 mm to (24.9, 3.81)
Routing:
- net N$7: track 4.97 -> 3.99 mm
